File: PCB/Version 1/ESP32-C3.kicad_pcb (KiCad board)
At the start: 2 copper layers, 28.3 x 28.7 mm, 50 parts, among them J1 HCZZ0039-3, J2 DPS_PPS_Right_Angle, SW1 TS-1187A-B-A-B, SW2 TS-1187A-B-A-B, U1 USB-C-16P-SMD, U2 BQ24073RGTR, U3 ESP32-C3, U5 WL9003S5-33, Y1 40MHz_S3240000151040

Commit message: Update firmware, hardware documentation, and public README
Other:
- board text added: "V1 W-Charger 06.2024"
- board text removed: "A.S. V1 W-Charger 06.2024"
Changed lines of the file:
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@@
 		(layer "Edge.Cuts")
 	)
-	(gr_text "A.S.     V1\nW-Charger\n 06.2024"
+	(gr_text "         V1\nW-Charger\n 06.2024"
 		(at 148.9 85.9 0)
 		(layer "B.SilkS" knockout)
