File: PCB/Version 3/ESP32-C3-V3.kicad_pcb (KiCad board)
At the start: 4 copper layers, 27.7 x 24.3 mm, 49 parts, among them J1 PH1257-WT-04, J2 DPS_PPS, Q1 SI2301CDS-T1-GE3, SW2 TS-1187A-B-A-B, U1 USB-C-16P-SMD, U2 DS8561-33S5, U3 ESP32-C3, U4 TC4056A, U5 SKCL3130ME, Y1 40MHz_S3240000151040

Commit message: Update firmware, hardware documentation, and public README
Other:
- board text added: "V3 W-Charger 07.24"
- board text removed: "A.S. V3 W-Charger 07.24"
Changed lines of the file:
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@@
 		)
 	)
-	(gr_text "A.S.            V3\nW-Charger  07.24"
+	(gr_text "                V3\nW-Charger  07.24"
 		(at 153.7 93.3 270)
 		(layer "B.SilkS" knockout)
