File: PCB/Version 4/ESP32-C3-V4/ESP32-C3-V4.kicad_sch (KiCad schematic)
At the start: 31 parts, among them J1 M1257RS-04P, Q3 SI2301CDS-T1-GE3, Q4 2N7002, Q5 SI2301CDS-T1-GE3, SW1 TS-1088-AR02016, U1 USB-C-16P-SMD, U3 ESP32-C3

Commit message: Update Version 4 PCB and production outputs
Parts:
- removed AE1: KH-3216-H0209, RF_Antenna:Texas_SWRA117D_2.4GHz_Left, symbol ESP32-C3_Bib:KH-3216-H0209
- removed C1, C11, C5, C7: 100n_0402_X7R_16V, Capacitor_SMD:C_0402_1005Metric, symbol capacitor_smd_standard:100n_0402_X7R_16V
- removed C2: 10u_0402_X5R_6V3, Capacitor_SMD:C_0402_1005Metric, symbol capacitor_smd_standard:10u_0402_X5R_6V3
- removed C3, C6: 3p3_0402_C0G_50V, Capacitor_SMD:C_0402_1005Metric, symbol ESP32-C3_Bib:3p3_0402_C0G_50V
- removed L1: 2n2H_0403_500mA, Resistor_SMD:R_0402_1005Metric, symbol ESP32-C3_Bib:2n2H_0403_500mA
- removed R8: 330k_0603, Resistor_SMD:R_0603_1608Metric, symbol resistor_smd_standard:330k_0603
- removed SW1: TS-1088-AR02016, footprints:SW_TS-1088_XNP, symbol 2026-08-07_10-44-14:TS-1088-AR02016
- removed U3: ESP32-C3, Package_DFN_QFN:QFN-32-1EP_5x5mm_P0.5mm_EP3.7x3.7mm, symbol ESP32-C3:ESP32-C3
- added AE1: ANT3216LL00R2400A, Resistor_SMD:R_1206_3216Metric, symbol ESP32-C3_Bib:ANT3216LL00R2400A_2_4GHz_Antenne
- added C1, C2: 20p_0402_C0G_50V, Capacitor_SMD:C_0402_1005Metric, symbol Lil-Lib:20p_0402_C0G_50V
- added C16, C17, C21, C22, C23: 100n_0402_X7R_16V, Capacitor_SMD:C_0402_1005Metric, symbol capacitor_smd_standard:100n_0402_X7R_16V
- added C18, C19: 3p3_0402_C0G_50V, Capacitor_SMD:C_0402_1005Metric, symbol ESP32-C3_Bib:3p3_0402_C0G_50V
- added C20: 10u_0402_X5R_6V3, Capacitor_SMD:C_0402_1005Metric, symbol capacitor_smd_standard:10u_0402_X5R_6V3
- added L3: 2n2H_0403_500mA, Resistor_SMD:R_0402_1005Metric, symbol ESP32-C3_Bib:2n2H_0403_500mA
- added R11: 150k_0603, Resistor_SMD:R_0603_1608Metric, symbol resistor_smd_standard:150k_0603
- added R8: 100k_0402, Resistor_SMD:R_0402_1005Metric, symbol resistor_smd_standard:100k_0402
- added SW2: TS-1088-AR02016, footprints:SW_TS-1088_XNP, symbol 2026-08-07_10-44-14:TS-1088-AR02016
- added U2: ESP32-C3, Package_DFN_QFN:QFN-32-1EP_5x5mm_P0.5mm_EP3.7x3.7mm, symbol MCU_Espressif:ESP32-C3
- added Y1: 40MHz_S3240000151040, Crystal:Crystal_SMD_3225-4Pin_3.2x2.5mm, symbol ESP32-C3_Bib:40MHz_S3240000151040
- J1: LCSC C541828 -> C2939383
Connections:
- net +3.3V: now also Q5.2 (S), C16.1, C17.1, C20.2, C21.2, C22.2, C23.1, R8.1, U2.11 (VDD3P3_RTC), U2.17 (VDD3P3_CPU), U2.18 (VDD_SPI), U2.2 (VDD3P3), U2.3 (VDD3P3), U2.31 (VDDA), U2.32 (VDDA); no longer Q5.3 (D)
- net +BATT: now also Q3.2 (S); no longer Q3.3 (D)
- net ADC: now also U2.8 (GPIO3)
- net CHIP_EN: now also U2.7 (CHIP_EN)
- net EXTI: now also U2.6 (GPIO2)
- net GND: now also C1.1, C16.2, C17.2, C18.2, C19.2, C2.1, C20.1, C21.1, C22.1, C23.2, R11.2, SW2.1, U2.33 (GND), Y1.2 (GND), Y1.4 (GND)
- net GPIO8: now also U2.14 (GPIO8)
- net MCU_SCL: now also U2.9 (MTMS)
- net MCU_SDA: now also U2.10 (MTDI)
- net SENSOR_PWR_EN: now also U2.16 (GPIO10)
- net USB_D+: now also U2.26 (GPIO19)
- net USB_D-: now also U2.25 (GPIO18)
- net at R13.2, R17.1: now also R11.1
- net at J1.1 (Pin_1), R10.2, R9.2: now also Q5.3 (D); no longer Q5.2 (S)
- net at R13.1: now also Q3.3 (D); no longer Q3.2 (S)
- net ADC_On_Off renamed ADC_EN
- net ADC_EN: now also U2.12 (MTCK)
- new net: C2.2, U2.30 (XTAL_P), Y1.1 (OSC1)
- new net: C1.2, U2.29 (XTAL_N), Y1.3 (OSC2)
- new net: R8.2, SW2.2, U2.15 (GPIO9)
- new net: AE1.1 (A), C18.1, L3.1
- new net: C19.1, L3.2, U2.1 (LNA_IN)
- no-connect marks 24 -> 21
Other:
- note added: "2,75 V_in = 1,65 V_out"
- note added: "4,2 V_in = 2,52 V_out"
- moved on the sheet: Q3, Q5, R2, R3
