File: PCB/Version 4/ESP32-C3-V4/charger.kicad_sch (KiCad schematic)
At the start: 21 parts, among them J2 DPS_PPS, Q1 SI2301CDS-T1-GE3, U4 TC4056A, U5 SKCL3130ME, U6 TPS63900DSKR

Commit message: Update Version 4 PCB and production outputs
Parts:
- removed C12: 10u_0402_X5R_6V3, Capacitor_SMD:C_0402_1005Metric, symbol capacitor_smd_standard:10u_0402_X5R_6V3
- removed D3: 0603_WHITE, LED_SMD:LED_0603_1608Metric, symbol led:0603_GREEN
- removed D4: 1N5819WS(Basic), Diode_SMD:D_SOD-323_HandSoldering, symbol 1_diodes:1N5819WS(Basic)
- removed J2: DPS_PPS, Connector_JST:JST_PH_B2B-PH-K_1x02_P2.00mm_Vertical, symbol DPS_connectors:DPS_PPS
- removed R12: 330k_0603, Resistor_SMD:R_0603_1608Metric, symbol resistor_smd_standard:330k_0603
- removed U4: TC4056A, Package_SO:SOP-8_3.9x4.9mm_P1.27mm, symbol Lil-Lib:TC4056A
- added C25: 22u_0603_X5R_6V3, Capacitor_SMD:C_0603_1608Metric, symbol capacitor_smd_standard:22u_0603_X5R_6V3
- added D1: M7(Basic), Diode_SMD:D_SMA, symbol 1_diodes:M7(Basic)
- added D3: XL-1608UGC-04(Green), LED_SMD:LED_0603_1608Metric, symbol led:XL-1608UGC-04(Green 0603 ext)
- added J2: BatConnect2PSMD, Connector_JST:JST_PH_S2B-PH-SM4-TB_1x02-1MP_P2.00mm_Horizontal, symbol DPS_connectors:BatConnect2PSMD
- added R12: 33k_0402, Resistor_SMD:R_0402_1005Metric, symbol resistor_smd_standard:33k_0402
- added U3: TP4056-42-ESOP8, Package_SO:HTSOP-8-1EP_3.9x4.9mm_P1.27mm_EP2.4x3.2mm_ThermalVias, symbol Lil-Lib:TP4056-42-ESOP8
Connections:
- net +BATT: now also J2.2 (Pin_2), U3.5 (BAT)
- net Earth: now also J2.1 (Pin_1)
- net GND: now also C25.2, R12.2, U3.1 (TEMP), U3.3 (GND), U3.9 (EPAD)
- net VCC: now also D1.2 (A), R12.1, U3.4 (VCC), U3.8 (CE)
- net V_LDO: now also U6.1 (EN), U6.2 (SEL), C25.1, D1.1 (K)
- net at D2.1 (K): now also U3.7 (CHRG)
- net at R16.2: now also U3.2 (PROG)
- net at R20.1: now also D3.2 (A)
- new net: D3.1 (K), U3.6 (Full)
- no-connect marks 3 -> 1
Other:
- moved on the sheet: C13, C8, R4
